File: kicad/STM32F042F.sch (KiCad schematic (older format))
At the start: 11 parts, among them J2 SWD, J3 USB_B_Mini, U2 MCP1700-3302E_SOT89, U3 STM32F042F4Px

Commit message: Update STM32F042F.sch
Parts:
- R13, R4: value 100 -> 22
Changed lines of the file:
@@
 P 3250 4850
 F 0 "R13" H 3320 4896 50  0000 L CNN
-F 1 "100" H 3320 4805 50  0000 L CNN
+F 1 "22" H 3320 4805 50  0000 L CNN
 F 2 "Resistor_SMD:R_0805_2012Metric_Pad1.15x1.40mm_HandSolder" V 3180 4850 50  0001 C CNN
 F 3 "~" H 3250 4850 50  0001 C CNN
@@
 P 2900 4850
 F 0 "R4" H 2970 4896 50  0000 L CNN
-F 1 "100" H 2970 4805 50  0000 L CNN
+F 1 "22" H 2970 4805 50  0000 L CNN
 F 2 "Resistor_SMD:R_0805_2012Metric_Pad1.15x1.40mm_HandSolder" V 2830 4850 50  0001 C CNN
 F 3 "~" H 2900 4850 50  0001 C CNN
